File: DistBoard (WIP).kicad_sch (KiCad schematic)
At the start: 27 parts, among them J1 22-27-2021, J10 Conn_01x03, J11 Conn_01x03, J12 Conn_01x03, J13 Conn_01x03, J14 PPTC241LFBN-RC, J15 PPTC241LFBN-RC, J2 Conn_01x03, J3 Conn_01x03, J4 Conn_01x03, J5 Conn_01x03, J6 Conn_01x03, J7 Conn_01x03, J8 Conn_01x03, J9 Conn_01x03, U1 TLE2426CDR

Commit message: improved readability.
Connections:
- net AGND: no longer J12.3 (Pin_3)
Other:
- moved on the sheet: J2, J3, J4, J5, J6, J7, J8, J9
